File: rp2040_controller.kicad_pcb (KiCad board)
At the start: 2 copper layers, 16 x 52 mm, 36 parts, among them J1 10118193-0001LF, J2 Conn_01x02, SW1 PTS810_SJK_250_SMTR_LFS, U1 RP2040, U2 AP2112K-3.3TRG1, U3 W25Q16JVSSIQ, Y1 12MHz

Commit message: init
Parts:
- removed CR1: MBR120VLSFT1G, mbr120vlsft1g:MBR120VLSFT1G
- removed H2, H3, H4: MountingHole, MountingHole:MountingHole_2.1mm
- removed J2: Conn_01x02, custom:PinHeader_1x02_P2.54mm_Vertical_no-silk
- removed R6: DNP, Resistor_SMD:R_0603_1608Metric_Pad0.98x0.95mm_HandSolder
- removed R7: 1K, Resistor_SMD:R_0603_1608Metric_Pad0.98x0.95mm_HandSolder
- added J3: Conn_01x12, Connector_PinHeader_1.00mm:PinHeader_1x12_P1.00mm_Vertical, F.Cu at (94.1, 134.6)
- added REF**: SW_SPST_PTS810, Button_Switch_SMD:SW_SPST_PTS810, B.Cu at (105.5, 92.8)
- C1, C10, C11, C12, C14, C16, C2, C3, C4, C5, C6, C7, C8, C9: footprint Capacitor_SMD:C_0603_1608Metric_Pad1.08x0.95mm_HandSolder -> Capacitor_SMD_AKL:C_0603_1608Metric_Pad1.08x0.95mm
- C13, C15: value 27pF -> 12pF; footprint Capacitor_SMD:C_0603_1608Metric_Pad1.08x0.95mm_HandSolder -> Capacitor_SMD_AKL:C_0603_1608Metric_Pad1.08x0.95mm
- H1: footprint MountingHole:MountingHole_2.1mm -> ec_parts:keyboard_layout; moved to F.Cu
- J1: value 10118193-0001LF -> Conn_01x08_MountingPin; footprint 10118193-0001LF:FCI_10118193-0001LF_no-slot -> ec_parts:HRS_FH34SRJ-10S-0.5SH(50)
- R1, R3, R4, R5, R8, R9: footprint Resistor_SMD:R_0603_1608Metric_Pad0.98x0.95mm_HandSolder -> Resistor_SMD_AKL:R_0603_1608Metric_Pad0.98x0.95mm_HandSolder
- SW1: value PTS810_SJK_250_SMTR_LFS -> RotaryEncoder_Switch; footprint PTS810 SJK 250 SMTR LFS:PTS810 SJK 250 SMTR LFS -> ec_parts:EVQWGD001_without_cut; moved to F.Cu
- U3: value W25Q16JVSSIQ -> W25Q64JV; footprint W25Q16JVSSIQ:SOIC127P790X216-8N -> Package_SON:WSON-8-1EP_6x5mm_P1.27mm_EP3.4x4mm
- Y1: value 12MHz -> XYDBPCNANF-12MHZ; footprint abls7m:ABLS7M2-16.000MHZ-D-2Y-T -> Crystal_AKL:Crystal_SMD_2520-4Pin_2.5x2.0mm
- moved SW1 33.5 mm to (99.6, 125.9)
- moved H1 27.3 mm to (100.0, 104.7), turned to 0 degrees
- moved C16 26.3 mm to (99.4, 107.4), turned to -90 degrees
- moved C14 22.3 mm to (94.9, 111.1)
- moved U2 22.3 mm to (94.9, 108.4)
- moved U3 21.3 mm to (103.6, 108.5), turned to 180 degrees
- moved C6 20.3 mm to (95.5, 105.7), turned to 180 degrees
- moved R3 19.5 mm to (97.8, 108.4)
- moved R9 19.5 mm to (106.2, 113.0)
- moved C10 16.9 mm to (95.2, 113.9), turned to 180 degrees
- moved C11 16.3 mm to (99.0, 126.2), turned to -90 degrees
- moved C1 16.0 mm to (102.5, 113.0)
- moved C12 16.0 mm to (98.0, 113.0)
- moved C9 16.0 mm to (104.0, 113.0)
- moved R4 16.0 mm to (101.0, 113.0)
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Connections:
- C15 pad 1: Net-(C15-Pad1) -> /XOUT
- J1 pad 1: /VBUS -> /VSYS
- J1 pad 2: /USB_N -> /USB_P
- J1 pad 3: /USB_P -> /USB_N
- J1 pad 5: GND -> unconnected-(J1-Pad5)
- R4 pad 1: /USB_P -> /USB_N
- R5 pad 1: /USB_N -> /USB_P
- U1 pad 11: unconnected-(U1-Pad11) -> /GPIO8
- U1 pad 12: unconnected-(U1-Pad12) -> /GPIO9
- U1 pad 13: unconnected-(U1-Pad13) -> /GPIO10
- U1 pad 14: unconnected-(U1-Pad14) -> /GPIO11
- U1 pad 15: unconnected-(U1-Pad15) -> /GPIO12
- U1 pad 16: unconnected-(U1-Pad16) -> /GPIO13
- U1 pad 17: unconnected-(U1-Pad17) -> /GPIO14
- U1 pad 18: unconnected-(U1-Pad18) -> /GPIO15
- U1 pad 2: unconnected-(U1-Pad2) -> /GPIO0
- U1 pad 27: unconnected-(U1-Pad27) -> /GPIO16
- U1 pad 28: unconnected-(U1-Pad28) -> /GPIO17
- U1 pad 29: unconnected-(U1-Pad29) -> /GPIO18
- U1 pad 3: unconnected-(U1-Pad3) -> /GPIO1
- U1 pad 30: unconnected-(U1-Pad30) -> /GPIO19
- U1 pad 31: unconnected-(U1-Pad31) -> /GPIO20
- U1 pad 32: unconnected-(U1-Pad32) -> /GPIO21
- U1 pad 34: unconnected-(U1-Pad34) -> /GPIO22
- U1 pad 35: unconnected-(U1-Pad35) -> /GPIO23
- U1 pad 36: unconnected-(U1-Pad36) -> /GPIO24
- U1 pad 4: unconnected-(U1-Pad4) -> /GPIO2
- U1 pad 46: Net-(R5-Pad2) -> Net-(R4-Pad2)
- U1 pad 47: Net-(R4-Pad2) -> Net-(R5-Pad2)
- U1 pad 5: unconnected-(U1-Pad5) -> /GPIO3
- U1 pad 6: unconnected-(U1-Pad6) -> /GPIO4
- U1 pad 7: unconnected-(U1-Pad7) -> /GPIO5
- U1 pad 8: unconnected-(U1-Pad8) -> /GPIO6
- U1 pad 9: unconnected-(U1-Pad9) -> /GPIO7
- Y1 pad 1: /XIN -> /XOUT
- Y1 pad 2: Net-(C15-Pad1) -> GND
Routing:
- net +3V3: track 125.5 -> 47.9 mm, vias 2 -> 6
- net /GPIO5: track 0.00 -> 51.5 mm, vias 0 -> 1
- net /USB_BOOT: track 37.1 -> 0.00 mm, vias 3 -> 0
- net /GPIO0: track 0.00 -> 26.3 mm, vias 0 -> 1
- net /GPIO4: track 0.00 -> 26.0 mm, vias 0 -> 1
- net /GPIO2: track 0.00 -> 25.9 mm, vias 0 -> 1
- net /GPIO1: track 0.00 -> 25.2 mm, vias 0 -> 1
- net /GPIO7: track 0.00 -> 25.0 mm, vias 0 -> 1
- net /GPIO3: track 0.00 -> 17.8 mm, vias 0 -> 1
- net /RUN: track 20.6 -> 3.94 mm, vias 2 -> 1
- net /USB_N: track 16.0 -> 0.00 mm
- net /USB_P: track 16.0 -> 0.00 mm
- net /QSPI_SD0: track 23.0 -> 10.3 mm, vias 2 -> 3
- net /QSPI_SCK: track 22.1 -> 10.1 mm
- net /QSPI_SD3: track 19.6 -> 9.33 mm
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Other:
- board size 16 x 52 mm -> 66.8 x 15.3 mm
- copper layers 2 -> 4
- board text removed: "10"
- board text removed: "11"
- board text removed: "12"
- board text removed: "13"
- board text removed: "14"
- board text removed: "15"
- board text removed: "16"
- board text removed: "17"
- board text removed: "18"
- board text removed: "19"
- board text removed: "2"
- board text removed: "20"
- board text removed: "21"
- board text removed: "22"
- board text removed: "26"
- board text removed: "27"
- board text removed: "28"
- board text removed: "3"
- board text removed: "3V3"
- board text removed: "4"
- board text removed: "5"
- board text removed: "6"
- board text removed: "7"
- board text removed: "8"
- board text removed: "9"
- board text removed: "AREF"
- board text removed: "BTSEL"
- board text removed: "CLK"
- board text removed: "DIO"
- board text removed: "EN"
- board text removed: "GND"
- board text removed: "RESET"
- board text removed: "RPi Pico Debugger Shoe"
- board text removed: "RUN"
- board text removed: "SHOE SWD"
- board text removed: "TGT_TX"
- board text removed: "VBUS"
- board text removed: "VSYS"
- board text removed: "v02"

Commit message: temp
Parts:
- removed the REF** at (105.5, 92.8)
- removed SW1: RotaryEncoder_Switch, ec_parts:EVQWGD001_without_cut
- added REF**: Molex_Pico-EZmate_78171-0005_1x05-1MP_P1.20mm_Vertical, Connector_Molex:Molex_Pico-EZmate_78171-0005_1x05-1MP_P1.20mm_Vertical, F.Cu at (100.4, 102.2)
- C1, C10, C11, C12, C13, C14, C15, C16, C2, C3, C4, C5, C6, C7, C8, C9, J1, R1, R3, R4, R5, R8, R9, U1, U2, U3, Y1: moved to F.Cu
- J3: footprint Connector_PinHeader_1.00mm:PinHeader_1x12_P1.00mm_Vertical -> ec_parts:ed_pad_1x12_P1.27mm
- moved J1 50.8 mm to (104.8, 143.9)
- moved C3 13.7 mm to (93.6, 123.9), turned to 180 degrees
- moved C2 13.6 mm to (93.6, 120.2), turned to 180 degrees
- moved C6 12.3 mm to (107.5, 108.4), turned to 90 degrees
- moved R9 11.9 mm to (94.8, 116.4)
- moved U2 11.8 mm to (106.0, 112.4), turned to -90 degrees
- moved C14 11.6 mm to (105.7, 115.4), turned to 180 degrees
- moved C7 11.0 mm to (105.8, 120.4), turned to 0 degrees
- moved C8 11.0 mm to (105.8, 118.8), turned to 0 degrees
- moved C10 11.0 mm to (105.7, 117.2), turned to 0 degrees
- moved C13 10.9 mm to (95.3, 129.5)
- moved R3 10.3 mm to (108.0, 109.7), turned to 180 degrees
- moved R8 10.2 mm to (95.7, 108.1), turned to 0 degrees
- moved C5 9.50 mm to (105.8, 122.9), turned to 0 degrees
- moved C9 7.73 mm to (97.0, 116.4)
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Connections:
- J3 pad 1: unconnected-(J3-Pad1) -> +3V3
- J3 pad 10: unconnected-(J3-Pad10) -> /GPIO14
- J3 pad 12: unconnected-(J3-Pad12) -> GND
- J3 pad 2: unconnected-(J3-Pad2) -> /GPIO18
- J3 pad 3: unconnected-(J3-Pad3) -> /GPIO17
- J3 pad 4: unconnected-(J3-Pad4) -> /GPIO16
- J3 pad 5: unconnected-(J3-Pad5) -> /GPIO26/ADC0
- J3 pad 6: unconnected-(J3-Pad6) -> /GPIO27/ADC1
- J3 pad 7: unconnected-(J3-Pad7) -> /GPIO28/ADC2
- J3 pad 8: unconnected-(J3-Pad8) -> /GPIO29/ADC3
- J3 pad 9: unconnected-(J3-Pad9) -> /GPIO15
- R4 pad 1: /USB_N -> /USB_P
- R5 pad 1: /USB_P -> /USB_N
- U1 pad 38: /GPIO26/ADC3 -> /GPIO26/ADC0
- U1 pad 39: /GPIO27/ADC3 -> /GPIO27/ADC1
- U1 pad 40: /GPIO28/ADC3 -> /GPIO28/ADC2
- U1 pad 46: Net-(R4-Pad2) -> Net-(R5-Pad2)
- U1 pad 47: Net-(R5-Pad2) -> Net-(R4-Pad2)
Routing:
- net /GPIO5: track 51.5 -> 0.00 mm, vias 1 -> 0
- net /GPIO0: track 26.3 -> 0.00 mm, vias 1 -> 0
- net /GPIO4: track 26.0 -> 0.00 mm, vias 1 -> 0
- net /GPIO2: track 25.9 -> 0.00 mm, vias 1 -> 0
- net /GPIO1: track 25.2 -> 0.00 mm, vias 1 -> 0
- net /GPIO7: track 25.0 -> 0.00 mm, vias 1 -> 0
- net /GPIO3: track 17.8 -> 0.00 mm, vias 1 -> 0
- net /GPIO26/ADC0: track 0.00 -> 8.21 mm, vias 0 -> 1
- net /GPIO29/ADC3: track 0.00 -> 5.46 mm, vias 0 -> 1
- net +3V3: track 47.9 -> 43.9 mm
- net /GPIO16: track 0.00 -> 3.70 mm
- net /VSYS: track 3.59 -> 0.00 mm
- net Net-(R3-Pad2): track 1.73 -> 5.33 mm
- net /GPIO27/ADC1: track 0.00 -> 3.55 mm, vias 0 -> 1
- net /GPIO17: track 0.00 -> 3.24 mm
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Other:
- board text removed: "TGT_RX"

Commit message: temp
Parts:
- removed H1: MountingHole, ec_parts:keyboard_layout
- removed REF**: Molex_Pico-EZmate_78171-0005_1x05-1MP_P1.20mm_Vertical, Connector_Molex:Molex_Pico-EZmate_78171-0005_1x05-1MP_P1.20mm_Vertical
- added J2: Conn_01x10, Connector_PinHeader_2.54mm:PinHeader_1x11_P2.54mm_Vertical, B.Cu at (108.0, 107.6)
- added J4: Conn_01x10, Connector_PinHeader_2.54mm:PinHeader_1x11_P2.54mm_Vertical, B.Cu at (92.0, 107.6)
- added J5: Conn_01x04, Connector_PinHeader_1.27mm:PinHeader_1x04_P1.27mm_Vertical, F.Cu at (91.3, 105.0)
- added R2: 27, Resistor_SMD_AKL:R_0603_1608Metric_Pad0.98x0.95mm_HandSolder, B.Cu at (100.5, 107.6)
- added R6: 27, Resistor_SMD_AKL:R_0603_1608Metric_Pad0.98x0.95mm_HandSolder, B.Cu at (102.0, 107.6)
- C1, C10, C11, C12, C13, C14, C15, C16, C2, C3, C4, C5, C6, C7, C8, C9, R1, R3, R4, R5, R8, R9, U1, U2, U3, Y1: moved to B.Cu
- J1: value Conn_01x08_MountingPin -> Conn_01x06_MountingPin
- moved J1 38.1 mm to (100.0, 106.1)
- moved C6 13.5 mm to (96.0, 115.5), turned to 180 degrees
- moved C3 12.2 mm to (105.4, 127.1), turned to -90 degrees
- moved C5 12.1 mm to (94.6, 127.5), turned to -90 degrees
- moved C2 12.0 mm to (105.4, 121.9), turned to 90 degrees
- moved C7 11.7 mm to (94.6, 123.9), turned to -90 degrees
- moved C8 11.3 mm to (94.6, 120.4), turned to 90 degrees
- moved R3 10.5 mm to (98.7, 114.6), turned to 90 degrees
- moved U2 10.1 mm to (95.9, 112.8), turned to 90 degrees
- moved C10 9.54 mm to (96.2, 118.2), turned to 90 degrees
- moved C13 9.37 mm to (104.5, 131.5)
- moved R8 9.28 mm to (104.7, 110.2)
- moved R1 9.23 mm to (94.6, 131.2)
- moved R9 9.06 mm to (101.4, 110.2), turned to 0 degrees
- moved C9 8.20 mm to (104.7, 119.1), turned to 0 degrees
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Connections:
- J1 pad 1: /VSYS -> unconnected-(J1-Pad1)
- J1 pad 2: /USB_P -> unconnected-(J1-Pad2)
- J1 pad 3: /USB_N -> GND
- J1 pad 4: unconnected-(J1-Pad4) -> /GPIO1
- J1 pad 5: unconnected-(J1-Pad5) -> /GPIO0
- J1 pad 6: unconnected-(J1-Pad6) -> /USB_P
- J1 pad 7: unconnected-(J1-Pad7) -> /USB_N
- J1 pad 8: GND -> /VSYS
- J1 pad MP: GND -> unconnected-(J1-PadMP)
- J3 pad 10: /GPIO14 -> /GPIO15
- J3 pad 11: unconnected-(J3-Pad11) -> /GPIO14
- J3 pad 12: GND -> /GPIO13
- J3 pad 2: /GPIO18 -> GND
- J3 pad 3: /GPIO17 -> /GPIO19
- J3 pad 4: /GPIO16 -> /GPIO18
- J3 pad 5: /GPIO26/ADC0 -> /GPIO17
- J3 pad 6: /GPIO27/ADC1 -> /GPIO16
- J3 pad 7: /GPIO28/ADC2 -> /GPIO26/ADC0
- J3 pad 8: /GPIO29/ADC3 -> /GPIO27/ADC1
- J3 pad 9: /GPIO15 -> /GPIO28/ADC2
Routing:
- net /SWDIO: track 0.00 -> 28.5 mm, vias 0 -> 1
- net /SWCLK: track 0.00 -> 27.1 mm, vias 0 -> 1
- net /RUN: track 3.67 -> 27.8 mm, vias 0 -> 1
- net /GPIO2: track 0.00 -> 21.8 mm, vias 0 -> 1
- net /GPIO0: track 0.00 -> 21.1 mm, vias 0 -> 2
- net /GPIO3: track 0.00 -> 19.3 mm, vias 0 -> 1
- net /GPIO1: track 0.00 -> 17.5 mm, vias 0 -> 2
- net /VSYS: track 0.00 -> 15.4 mm, vias 0 -> 1
- net /GPIO5: track 0.00 -> 15.1 mm, vias 0 -> 1
- net /USB_P: track 0.00 -> 13.4 mm, vias 0 -> 2
- net /GPIO28/ADC2: track 2.62 -> 15.7 mm
- net /USB_N: track 0.00 -> 12.8 mm, vias 0 -> 2
- net /GPIO6: track 0.00 -> 12.7 mm
- net /GPIO25: track 0.00 -> 12.3 mm, vias 0 -> 1
- net /GPIO7: track 0.00 -> 10.6 mm
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- added copper zone on B.Cu, net +3V3
- added copper zone on In2.Cu, net +3V3
- added copper zone on B.Cu, net /VSYS
- added copper zone on F.Cu, net /VSYS
Other:
- board size 66.8 x 15.3 mm -> 19 x 52 mm
- board text added: "BTSEL"

Commit message: v0.1
Parts:
- added J6: Molex Pico Ezmate 1x04 or 1x06, ec_parts:Molex_Pico-EZmate_1.2mm_04_or_06, F.Cu at (100.0, 76.7)
- J1: value Conn_01x06_MountingPin -> FFC connector; footprint ec_parts:HRS_FH34SRJ-10S-0.5SH(50) -> ec_parts:HRS_FH34SRJ-08S-0.5SH(50)
- J2: value Conn_01x10 -> Right; footprint Connector_PinHeader_2.54mm:PinHeader_1x11_P2.54mm_Vertical -> ec_parts:Right_PinHeader_1x11_P2.54mm_Vertical
- J3: value Conn_01x12 -> Bottom pin pads; footprint ec_parts:ed_pad_1x12_P1.27mm -> ec_parts:ec_pad_1x15_P1.27mm
- J4: value Conn_01x10 -> Left; footprint Connector_PinHeader_2.54mm:PinHeader_1x11_P2.54mm_Vertical -> ec_parts:Left_PinHeader_1x12_P2.54mm_Vertical
- J5: footprint Connector_PinHeader_1.27mm:PinHeader_1x04_P1.27mm_Vertical -> ec_parts:TestPinHeader_1x03_P1.27mm_Vertical
- moved J5 38.8 mm to (107.4, 69.7), turned to -90 degrees
- moved J4 37.9 mm to (92.0, 69.7)
- moved C7 35.9 mm to (94.6, 88.1)
- moved C8 35.8 mm to (94.6, 84.7)
- moved C2 35.7 mm to (105.4, 86.3)
- moved C13 35.4 mm to (104.4, 96.2)
- moved C1 35.4 mm to (102.2, 82.9)
- moved C10 35.4 mm to (96.2, 82.9)
- moved C12 35.4 mm to (97.8, 82.9)
- moved C14 35.4 mm to (98.8, 75.7)
- moved C16 35.4 mm to (95.8, 74.4)
- moved C9 35.4 mm to (104.7, 83.8)
- moved R4 35.4 mm to (100.8, 82.9)
- moved R5 35.4 mm to (99.2, 82.9)
- moved U3 35.4 mm to (103.0, 78.3)
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Connections:
- J1 pad 1: unconnected-(J1-Pad1) -> GND
- J1 pad 2: unconnected-(J1-Pad2) -> /GPIO3
- J1 pad 3: GND -> /GPIO2
- J1 pad MP: unconnected-(J1-PadMP) -> GND
- J2 pad 10: /GPIO11 -> /GPIO10
- J2 pad 3: /GPIO5 -> /GPIO4
- J2 pad 4: /GPIO6 -> /GPIO5
- J2 pad 5: /GPIO7 -> /GPIO6
- J2 pad 6: /GPIO8 -> /GPIO7
- J2 pad 8: /GPIO9 -> /GPIO8
- J2 pad 9: /GPIO10 -> /GPIO9
- J3 pad 1: +3V3 -> GND
- J3 pad 10: /GPIO15 -> /GPIO14
- J3 pad 11: /GPIO14 -> /GPIO13
- J3 pad 12: /GPIO13 -> /GPIO12
- J3 pad 13: /GPIO12 -> /GPIO11
- J3 pad 14: GND -> +3V3
- J3 pad 15: +3V3 -> GND
- J3 pad 2: GND -> +3V3
- J4 pad 1: /RUN -> /VSYS
- J4 pad 10: /GPIO20 -> /GPIO21
- J4 pad 11: +3V3 -> /GPIO20
- J4 pad 2: GND -> /RUN
- J4 pad 3: /GPIO29/ADC3 -> GND
- J4 pad 4: /GPIO25 -> /GPIO29/ADC3
- J4 pad 5: /GPIO24 -> /GPIO25
- J4 pad 6: /GPIO23 -> /GPIO24
- J4 pad 7: GND -> /GPIO23
- J4 pad 8: /GPIO22 -> GND
- J4 pad 9: /GPIO21 -> /GPIO22
- J5 pad 1: /SWDIO -> /SWCLK
- J5 pad 3: /SWCLK -> /SWDIO
Routing:
- net /GPIO4: track 0.00 -> 14.6 mm
- net /VSYS: track 15.4 -> 4.56 mm, vias 1 -> 2
- net /GPIO19: track 0.00 -> 9.51 mm
- net /GPIO15: track 9.07 -> 0.00 mm, vias 1 -> 0
- net GND: track 2.39 -> 9.96 mm, vias 0 -> 17
- net /GPIO1: track 17.5 -> 24.1 mm, vias 2 -> 3
- net /SWCLK: track 27.1 -> 32.4 mm
- net /GPIO3: track 19.3 -> 24.3 mm
- net +3V3: track 34.9 -> 39.5 mm, vias 11 -> 12
- net /GPIO11: track 5.39 -> 8.95 mm
- net /GPIO8: track 9.91 -> 6.85 mm
- net /USB_P: track 13.4 -> 10.6 mm, vias 2 -> 1
- net /GPIO5: track 15.1 -> 12.6 mm, vias 1 -> 0
- net /SWDIO: track 28.5 -> 30.7 mm
- net /GPIO6: track 12.7 -> 10.6 mm, vias 0 -> 1
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- added copper zone on B.Cu, net GND
- added copper zone on F.Cu, net GND
- added copper zone on In1.Cu, net GND
- added copper zone on In2.Cu, net GND
Other:
- board size 19 x 52 mm -> 19 x 31.5 mm

Commit message: v0.2
Parts:
- removed J2: Right, ec_parts:Right_PinHeader_1x11_P2.54mm_Vertical
- removed J3: Bottom pin pads, ec_parts:ec_pad_1x15_P1.27mm
- removed J4: Left, ec_parts:Left_PinHeader_1x12_P2.54mm_Vertical
- removed J5: Conn_01x04, ec_parts:TestPinHeader_1x03_P1.27mm_Vertical
- removed J6: Molex Pico Ezmate 1x04 or 1x06, ec_parts:Molex_Pico-EZmate_1.2mm_04_or_06
- removed R2, R6: 27, Resistor_SMD_AKL:R_0603_1608Metric_Pad0.98x0.95mm_HandSolder
- J1: value FFC connector -> rp2040_controller; footprint ec_parts:HRS_FH34SRJ-08S-0.5SH(50) -> ec_parts:rp2040_controller
- moved J1 14.5 mm to (100.0, 85.2), turned to 0 degrees
Connections:
- J1 pad 1: GND -> /SWCLK
- J1 pad 2: /GPIO3 -> /VSYS
- J1 pad 3: /GPIO2 -> /USB_N
- J1 pad 4: /GPIO1 -> /USB_P
- J1 pad 6: /USB_P -> /GPIO1
- J1 pad 7: /USB_N -> +3V3
- J1 pad 8: /VSYS -> /USB_BOOT
Routing:
- net /GPIO29/ADC3: track 12.8 -> 0.00 mm, vias 1 -> 0
- net /GPIO25: track 12.4 -> 0.00 mm
- net /GPIO3: track 24.3 -> 13.7 mm, vias 1 -> 0
- net /SWCLK: track 32.4 -> 23.5 mm
- net /GPIO2: track 21.9 -> 15.9 mm
- net +3V3: track 39.5 -> 33.9 mm, vias 12 -> 11
- net /GPIO1: track 24.1 -> 18.8 mm, vias 3 -> 1
- net GND: track 9.96 -> 15.2 mm, vias 17 -> 30
- net /RUN: track 28.6 -> 23.9 mm
- net /SWDIO: track 30.7 -> 26.4 mm
- net /GPIO7: track 10.4 -> 7.38 mm, vias 1 -> 0
- net /GPIO24: track 10.5 -> 7.65 mm
- net /GPIO0: track 21.1 -> 18.2 mm, vias 2 -> 1
- net /GPIO8: track 6.85 -> 9.33 mm
- net /GPIO23: track 8.31 -> 6.09 mm
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Other:
- board size 19 x 31.5 mm -> 19 x 29.1 mm

Commit message: v0.3
Parts:
- added R2: 400, Resistor_SMD_AKL:R_0603_1608Metric_Pad0.98x0.95mm_HandSolder, B.Cu at (94.7, 82.9)
- U2: value AP2112K-3.3TRG1 -> AP2112K-3.3; footprint ap2112:AP2112K-3.3TRG1 -> Package_TO_SOT_SMD_AKL:SOT-23-5
- moved C8 0.91 mm to (95.2, 85.3), turned to 180 degrees
Connections:
- C8 pad 1: +3V3 -> /AVDD
- J1 pad 39: /GPIO2 -> GND
- J1 pad 40: /RUN -> /GPIO2
- J1 pad 41: GND -> /RUN
- J1 pad 7: +3V3 -> /USB_BOOT
- J1 pad 8: /USB_BOOT -> /GPIO3
- J1 pad 9: /GPIO3 -> +3V3
- U1 pad 43: +3V3 -> /AVDD
- Y1 pad 2: GND -> unconnected-(Y1-Pad2)
Routing:
- net /AVDD: track 0.00 -> 4.03 mm
- net GND: track 15.2 -> 12.6 mm
- net /GPIO0: track 18.2 -> 15.9 mm
- net /RUN: track 23.9 -> 25.9 mm
- net +3V3: track 33.9 -> 32.1 mm, vias 11 -> 13
- net /GPIO1: track 18.8 -> 20.3 mm
- net /SWDIO: track 26.4 -> 25.0 mm, vias 1 -> 2
- net /GPIO19: track 10.4 -> 9.18 mm
- net /GPIO3: track 13.7 -> 14.8 mm
- net /USB_BOOT: track 3.36 -> 2.36 mm
- net /GPIO28/ADC2: track 15.7 -> 16.5 mm
- net /GPIO2: track 15.9 -> 16.7 mm
- net /GPIO11: track 8.45 -> 9.20 mm
- net /GPIO27/ADC1: track 13.8 -> 14.6 mm
- net /SWCLK: track 23.5 -> 24.2 mm, vias 1 -> 2
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Other:
- board size 19 x 29.1 mm -> 19 x 29.2 mm

Commit message: temp
Parts:
- added J2: Conn_01x15, ec_parts:PinHeader_1x15_P1.27mm_Vertical, F.Cu at (91.1, 99.8)
- added J3: Conn_01x12, ec_parts:PinHeader_1x12_P2.54mm_Vertical, F.Cu at (107.8, 71.8)
- added J4: Conn_01x05, ec_parts:TestPinHeader_1x03_P1.27mm_Vertical, F.Cu at (100.0, 71.1)
- added J5: Conn_01x02, Connector_PinHeader_2.54mm:PinHeader_1x02_P2.54mm_Vertical, F.Cu at (97.3, 71.8)
- added J6: Conn_01x02, Connector_PinHeader_2.54mm:PinHeader_1x02_P2.54mm_Vertical, F.Cu at (105.2, 71.8)
- J1: value rp2040_controller -> Conn_01x12; footprint ec_parts:rp2040_controller -> ec_parts:PinHeader_1x12_P2.54mm_Vertical
- moved J1 15.5 mm to (92.2, 71.8)
- moved R1 0.30 mm to (94.9, 96.3)
- moved C5 0.10 mm to (94.4, 92.4)
- moved C8 0.10 mm to (95.3, 85.3)
Connections:
- J1 pad 1: /SWCLK -> /VSYS
- J1 pad 10: /GPIO5 -> /GPIO21
- J1 pad 11: /GPIO6 -> /GPIO20
- J1 pad 2: /VSYS -> /GPIO25
- J1 pad 3: /USB_N -> /RUN
- J1 pad 4: /USB_P -> GND
- J1 pad 5: /GPIO0 -> /GP_2/I2C_1_SDA/SPI_0_SCK
- J1 pad 6: /GPIO1 -> /GP_4/I2C_0_SDA/SPI_0_RX
- J1 pad 7: /USB_BOOT -> /GPIO24
- J1 pad 8: /GPIO3 -> /GPIO23
- J1 pad 9: +3V3 -> /GPIO22
- U1 pad 2: /GPIO0 -> /GPIO0/I2C0_SDA
- U1 pad 3: /GPIO1 -> /GPIO1/I2C0_SCL
- U1 pad 4: /GPIO2 -> /GP_2/I2C_1_SDA/SPI_0_SCK
- U1 pad 5: /GPIO3 -> /GP_3/I2C_1_SCL/SPI_0_TX 
- U1 pad 6: /GPIO4 -> /GP_4/I2C_0_SDA/SPI_0_RX
- U1 pad 7: /GPIO5 -> /GP_5/I2C_0_SCL/SPI_0_CS
- U1 pad 8: /GPIO6 -> /GP_6/I2C_1_SDA/SPI_0_SCK
- U1 pad 9: /GPIO7 -> /GP_7/I2C_1_SCL/SPI_0_TX
Routing:
- net /GPIO29/ADC3: track 0.00 -> 29.2 mm, vias 0 -> 2
- net /GPIO0/I2C0_SDA: track 0.00 -> 24.1 mm, vias 0 -> 2
- net /GPIO1: track 20.3 -> 0.00 mm, vias 1 -> 0
- net /GPIO25: track 0.00 -> 17.8 mm
- net /GPIO1/I2C0_SCL: track 0.00 -> 17.2 mm, vias 0 -> 1
- net /GPIO2: track 16.7 -> 0.00 mm, vias 1 -> 0
- net /GPIO0: track 15.9 -> 0.00 mm, vias 1 -> 0
- net /GPIO4: track 15.5 -> 0.00 mm, vias 1 -> 0
- net /GPIO3: track 14.8 -> 0.00 mm
- net /GP_2/I2C_1_SDA/SPI_0_SCK: track 0.00 -> 14.2 mm, vias 0 -> 1
- net /GP_4/I2C_0_SDA/SPI_0_RX: track 0.00 -> 13.8 mm, vias 0 -> 1
- net /GPIO5: track 11.8 -> 0.00 mm, vias 1 -> 0
- net /GP_3/I2C_1_SCL/SPI_0_TX : track 0.00 -> 9.91 mm, vias 0 -> 1
- net /GPIO6: track 9.89 -> 0.00 mm, vias 1 -> 0
- net /GP_5/I2C_0_SCL/SPI_0_CS: track 0.00 -> 7.72 mm
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- removed copper zone on B.Cu, net /VSYS
Other:
- board size 19 x 29.2 mm -> 19 x 29.5 mm
