File: rp2040_controller.kicad_sch (KiCad schematic)
At the start: 36 parts, among them J1 10118193-0001LF, J2 Conn_01x02, SW1 PTS810_SJK_250_SMTR_LFS, U1 RP2040, U2 AP2112K-3.3TRG1, U3 W25Q16JVSSIQ, Y1 12MHz

Commit message: init
Parts:
- removed C13, C15: 27pF, Capacitor_SMD:C_0603_1608Metric_Pad1.08x0.95mm_HandSolder, symbol Device:C
- removed CR1: MBR120VLSFT1G, mbr120vlsft1g:MBR120VLSFT1G, symbol rpi-pico-debugger-shoe-rescue:MBR120VLSFT1G-2021-05-12_00-49-18
- removed H2, H3, H4: MountingHole, MountingHole:MountingHole_2.1mm, symbol Mechanical:MountingHole
- removed J1: 10118193-0001LF, 10118193-0001LF:FCI_10118193-0001LF_no-slot, symbol rpi-pico-debugger-shoe-rescue:10118193-0001LF-10118193-0001LF
- removed J2: Conn_01x02, custom:PinHeader_1x02_P2.54mm_Vertical_no-silk, symbol Connector_Generic:Conn_01x02
- removed R6: DNP, Resistor_SMD:R_0603_1608Metric_Pad0.98x0.95mm_HandSolder, symbol Device:R
- removed R7: 1K, Resistor_SMD:R_0603_1608Metric_Pad0.98x0.95mm_HandSolder, symbol Device:R
- removed SW1: PTS810_SJK_250_SMTR_LFS, PTS810 SJK 250 SMTR LFS:PTS810 SJK 250 SMTR LFS, symbol rpi-pico-debugger-shoe-rescue:PTS810_SJK_250_SMTR_LFS-2021-05-12_02-12-02
- removed U3: W25Q16JVSSIQ, W25Q16JVSSIQ:SOIC127P790X216-8N, symbol rpi-pico-debugger-shoe-rescue:W25Q16JVSSIQ-W25Q16JVSSIQ
- removed Y1: 12MHz, abls7m:ABLS7M2-16.000MHZ-D-2Y-T, symbol Device:Crystal
- added C13, C15: 12pF, Capacitor_SMD_AKL:C_0603_1608Metric_Pad1.08x0.95mm, symbol Device:C_Small
- added J1: Conn_01x08_MountingPin, ec_parts:HRS_FH34SRJ-10S-0.5SH(50), symbol Connector_Generic_MountingPin:Conn_01x08_MountingPin
- added J3: Conn_01x12, Connector_PinHeader_1.00mm:PinHeader_1x12_P1.00mm_Vertical, symbol Connector_Generic:Conn_01x12
- added SW1: RotaryEncoder_Switch, ec_parts:EVQWGD001_without_cut, symbol Device:RotaryEncoder_Switch
- added U3: W25Q64JV, Package_SON:WSON-8-1EP_6x5mm_P1.27mm_EP3.4x4mm, symbol Memory_Flash_Extra:W25Q64JV
- added Y1: XYDBPCNANF-12MHZ, Crystal_AKL:Crystal_SMD_2520-4Pin_2.5x2.0mm, symbol Device:Crystal_GND24_Small
- C1, C10, C11, C12, C14, C16, C2, C3, C4, C5, C6, C7, C8, C9: footprint Capacitor_SMD:C_0603_1608Metric_Pad1.08x0.95mm_HandSolder -> Capacitor_SMD_AKL:C_0603_1608Metric_Pad1.08x0.95mm
- H1: footprint MountingHole:MountingHole_2.1mm -> ec_parts:keyboard_layout
- R1, R3, R8, R9: footprint Resistor_SMD:R_0603_1608Metric_Pad0.98x0.95mm_HandSolder -> Resistor_SMD_AKL:R_0603_1608Metric_Pad0.98x0.95mm_HandSolder
- R4: renamed from R5; footprint Resistor_SMD:R_0603_1608Metric_Pad0.98x0.95mm_HandSolder -> Resistor_SMD_AKL:R_0603_1608Metric_Pad0.98x0.95mm_HandSolder
- R5: renamed from R4; footprint Resistor_SMD:R_0603_1608Metric_Pad0.98x0.95mm_HandSolder -> Resistor_SMD_AKL:R_0603_1608Metric_Pad0.98x0.95mm_HandSolder
Connections:
- net +3V3: now also U3.8 (VDD)
- net GND: now also C13.2, C15.2, J1.8 (Pin_8), J1.MP (MountPin), U3.4 (GND), U3.9 (GND), Y1.2, Y1.4
- net QSPI_CS: now also U3.1 (~{CS})
- net QSPI_SCK: now also U3.6 (SCK)
- net QSPI_SD0: now also U3.5 (DI/IO0)
- net QSPI_SD1: now also U3.2 (DO/IO1)
- net QSPI_SD2: now also U3.3 (~{WP}/IO2)
- net QSPI_SD3: now also U3.7 (~{HOLD}/IO3)
- net USB_N: now also J1.3 (Pin_3)
- net USB_P: now also J1.2 (Pin_2)
- net VSYS: now also J1.1 (Pin_1)
- net XIN: now also C13.1, Y1.3
- net XOUT: now also C15.1, Y1.1
- net GPIO8: now reaches U1.11 (GPIO8)
- net GPIO9: now reaches U1.12 (GPIO9)
- net GPIO10: now reaches U1.13 (GPIO10)
- net GPIO11: now reaches U1.14 (GPIO11)
- net GPIO12: now reaches U1.15 (GPIO12)
- net GPIO13: now reaches U1.16 (GPIO13)
- net GPIO14: now reaches U1.17 (GPIO14)
- net GPIO15: now reaches U1.18 (GPIO15)
- net GPIO0: now reaches U1.2 (GPIO0)
- net GPIO16: now reaches U1.27 (GPIO16)
- net GPIO17: now reaches U1.28 (GPIO17)
- net GPIO18: now reaches U1.29 (GPIO18)
- net GPIO1: now reaches U1.3 (GPIO1)
- net GPIO19: now reaches U1.30 (GPIO19)
- net GPIO20: now reaches U1.31 (GPIO20)
- net GPIO21: now reaches U1.32 (GPIO21)
- net GPIO22: now reaches U1.34 (GPIO22)
- net GPIO23: now reaches U1.35 (GPIO23)
- net GPIO24: now reaches U1.36 (GPIO24)
- net GPIO2: now reaches U1.4 (GPIO2)
- net GPIO3: now reaches U1.5 (GPIO3)
- net GPIO4: now reaches U1.6 (GPIO4)
- net GPIO5: now reaches U1.7 (GPIO5)
- net GPIO6: now reaches U1.8 (GPIO6)
- net GPIO7: now reaches U1.9 (GPIO7)
- no-connect marks 2 -> 1
Other:
- note added: "12MHz"
- note removed: "LEDs"
- title: Raspberry Pi Pico Debugger Shoe -> RP2040 Controller
- moved on the sheet: C14, C16, C6, R3, U2

Commit message: temp
Parts:
- removed SW1: RotaryEncoder_Switch, ec_parts:EVQWGD001_without_cut, symbol Device:RotaryEncoder_Switch
- J1: value Conn_01x08_MountingPin -> Conn_01x06_MountingPin; symbol Connector_Generic_MountingPin:Conn_01x08_MountingPin -> Connector_Generic_MountingPin:Conn_01x06_MountingPin
- J3: footprint Connector_PinHeader_1.00mm:PinHeader_1x12_P1.00mm_Vertical -> ec_parts:ed_pad_1x12_P1.27mm
- renumbered R5 to R4, R4 to R5
Connections:
- net GPIO26/ADC3 is gone; now on net GPIO26/ADC0: U1.38 (GPIO26/ADC0)
- net GPIO27/ADC3 is gone; now on net GPIO27/ADC1: U1.39 (GPIO27/ADC1)
- net GPIO28/ADC3 is gone; now on net GPIO28/ADC2: U1.40 (GPIO28/ADC2)
- net +3V3: now also J3.1 (Pin_1)
- net GND: now also J1.6 (Pin_6), J3.12 (Pin_12); no longer J1.8 (Pin_8)
- net GPIO14: now also J3.10 (Pin_10)
- net GPIO15: now also J3.9 (Pin_9)
- net GPIO16: now also J3.4 (Pin_4)
- net GPIO17: now also J3.3 (Pin_3)
- net GPIO18: now also J3.2 (Pin_2)
- net GPIO29/ADC3: now also J3.8 (Pin_8)
- net GPIO26/ADC0: now reaches J3.5 (Pin_5)
- net GPIO27/ADC1: now reaches J3.6 (Pin_6)
- net GPIO28/ADC2: now reaches J3.7 (Pin_7)
Other:
- moved on the sheet: J3

Commit message: temp
Parts:
- removed H1: MountingHole, ec_parts:keyboard_layout, symbol Mechanical:MountingHole
- removed J1: Conn_01x06_MountingPin, ec_parts:HRS_FH34SRJ-10S-0.5SH(50), symbol Connector_Generic_MountingPin:Conn_01x06_MountingPin
- added J2, J4: Conn_01x10, Connector_PinHeader_2.54mm:PinHeader_1x11_P2.54mm_Vertical, symbol Connector_Generic:Conn_01x11
- added J5: Conn_01x04, Connector_PinHeader_1.27mm:PinHeader_1x04_P1.27mm_Vertical, symbol Connector_Generic:Conn_01x04
- added J?: Conn_01x06_MountingPin, ec_parts:HRS_FH34SRJ-10S-0.5SH(50), symbol Connector_Generic_MountingPin:Conn_01x08_MountingPin
- added R2, R6: 27, Resistor_SMD_AKL:R_0603_1608Metric_Pad0.98x0.95mm_HandSolder, symbol Device:R
- J3: symbol Connector_Generic:Conn_01x12 -> Connector_Generic:Conn_01x15
Connections:
- net +3V3: now also J3.15 (Pin_15), J2.11 (Pin_11), J2.2 (Pin_2), J4.11 (Pin_11), R2.2, R6.2
- net GND: now also J3.14 (Pin_14), J3.2 (Pin_2), J2.7 (Pin_7), J4.2 (Pin_2), J4.7 (Pin_7), J5.2 (Pin_2), J?.3 (Pin_3); no longer J3.12 (Pin_12)
- net GPIO0: now also J?.5 (Pin_5), R2.1
- net GPIO1: now also J?.4 (Pin_4), R6.1
- net GPIO10: now also J2.9 (Pin_9)
- net GPIO11: now also J2.10 (Pin_10)
- net GPIO12: now also J3.13 (Pin_13)
- net GPIO13: now also J3.12 (Pin_12)
- net GPIO14: now also J3.11 (Pin_11); no longer J3.10 (Pin_10)
- net GPIO15: now also J3.10 (Pin_10); no longer J3.9 (Pin_9)
- net GPIO16: now also J3.6 (Pin_6); no longer J3.4 (Pin_4)
- net GPIO17: now also J3.5 (Pin_5); no longer J3.3 (Pin_3)
- net GPIO18: now also J3.4 (Pin_4); no longer J3.2 (Pin_2)
- net GPIO19: now also J3.3 (Pin_3)
- net GPIO20: now also J4.10 (Pin_10)
- net GPIO21: now also J4.9 (Pin_9)
- net GPIO22: now also J4.8 (Pin_8)
- net GPIO23: now also J4.6 (Pin_6)
- net GPIO24: now also J4.5 (Pin_5)
- net GPIO25: now also J4.4 (Pin_4)
- net GPIO26/ADC0: now also J3.7 (Pin_7); no longer J3.5 (Pin_5)
- net GPIO27/ADC1: now also J3.8 (Pin_8); no longer J3.6 (Pin_6)
- net GPIO28/ADC2: now also J3.9 (Pin_9); no longer J3.7 (Pin_7)
- net GPIO29/ADC3: now also J4.3 (Pin_3); no longer J3.8 (Pin_8)
- net GPIO5: now also J2.3 (Pin_3)
- net GPIO6: now also J2.4 (Pin_4)
- net GPIO7: now also J2.5 (Pin_5)
- net GPIO8: now also J2.6 (Pin_6)
- net GPIO9: now also J2.8 (Pin_8)
- net RUN: now also J4.1 (Pin_1)
- net SWCLK: now also J5.3 (Pin_3)
- net SWDIO: now also J5.1 (Pin_1)
- net USB_BOOT: now also J2.1 (Pin_1)
- net USB_N: now also J?.7 (Pin_7)
- net USB_P: now also J?.6 (Pin_6)
- net VSYS: now also J5.4 (Pin_4), J?.8 (Pin_8)

Commit message: v0.1
Parts:
- added J6: Molex Pico Ezmate 1x04 or 1x06, ec_parts:Molex_Pico-EZmate_1.2mm_04_or_06, symbol Connector_Generic_MountingPin:Conn_01x06_MountingPin
- J1: renamed from J?; value Conn_01x06_MountingPin -> FFC connector; footprint ec_parts:HRS_FH34SRJ-10S-0.5SH(50) -> ec_parts:HRS_FH34SRJ-08S-0.5SH(50)
- J2: value Conn_01x10 -> Right; footprint Connector_PinHeader_2.54mm:PinHeader_1x11_P2.54mm_Vertical -> ec_parts:Right_PinHeader_1x11_P2.54mm_Vertical
- J3: value Conn_01x12 -> Bottom pin pads; footprint ec_parts:ed_pad_1x12_P1.27mm -> ec_parts:ec_pad_1x15_P1.27mm
- J4: value Conn_01x10 -> Left; footprint Connector_PinHeader_2.54mm:PinHeader_1x11_P2.54mm_Vertical -> ec_parts:Left_PinHeader_1x12_P2.54mm_Vertical; symbol Connector_Generic:Conn_01x11 -> Connector_Generic:Conn_01x12
- J5: footprint Connector_PinHeader_1.27mm:PinHeader_1x04_P1.27mm_Vertical -> ec_parts:TestPinHeader_1x03_P1.27mm_Vertical; symbol Connector_Generic:Conn_01x04 -> Connector_Generic:Conn_01x03
Connections:
- net +3V3: now also J3.14 (Pin_14), J3.2 (Pin_2); no longer J3.1 (Pin_1), J3.15 (Pin_15), J4.11 (Pin_11)
- net GND: now also J1.1 (Pin_1), J1.MP (MountPin), J3.1 (Pin_1), J3.15 (Pin_15), J4.12 (Pin_12), J4.3 (Pin_3), J4.8 (Pin_8), J6.4 (Pin_4), J6.MP (MountPin); no longer J1.3 (Pin_3), J3.14 (Pin_14), J3.2 (Pin_2), J4.2 (Pin_2), J4.7 (Pin_7)
- net GPIO0: now also J6.5 (Pin_5)
- net GPIO1: now also J6.6 (Pin_6)
- net GPIO10: now also J2.10 (Pin_10); no longer J2.9 (Pin_9)
- net GPIO11: now also J3.13 (Pin_13); no longer J2.10 (Pin_10)
- net GPIO12: now also J3.12 (Pin_12); no longer J3.13 (Pin_13)
- net GPIO13: now also J3.11 (Pin_11); no longer J3.12 (Pin_12)
- net GPIO14: now also J3.10 (Pin_10); no longer J3.11 (Pin_11)
- net GPIO15: no longer J3.10 (Pin_10)
- net GPIO2: now also J1.3 (Pin_3)
- net GPIO20: now also J4.11 (Pin_11); no longer J4.10 (Pin_10)
- net GPIO21: now also J4.10 (Pin_10); no longer J4.9 (Pin_9)
- net GPIO22: now also J4.9 (Pin_9); no longer J4.8 (Pin_8)
- net GPIO23: now also J4.7 (Pin_7); no longer J4.6 (Pin_6)
- net GPIO24: now also J4.6 (Pin_6); no longer J4.5 (Pin_5)
- net GPIO25: now also J4.5 (Pin_5); no longer J4.4 (Pin_4)
- net GPIO29/ADC3: now also J4.4 (Pin_4); no longer J4.3 (Pin_3)
- net GPIO3: now also J1.2 (Pin_2)
- net GPIO4: now also J2.3 (Pin_3)
- net GPIO5: now also J2.4 (Pin_4); no longer J2.3 (Pin_3)
- net GPIO6: now also J2.5 (Pin_5); no longer J2.4 (Pin_4)
- net GPIO7: now also J2.6 (Pin_6); no longer J2.5 (Pin_5)
- net GPIO8: now also J2.8 (Pin_8); no longer J2.6 (Pin_6)
- net GPIO9: now also J2.9 (Pin_9); no longer J2.8 (Pin_8)
- net RUN: now also J4.2 (Pin_2); no longer J4.1 (Pin_1)
- net SWCLK: now also J5.1 (Pin_1); no longer J5.3 (Pin_3)
- net SWDIO: now also J5.3 (Pin_3); no longer J5.1 (Pin_1)
- net USB_N: now also J6.2 (Pin_2)
- net USB_P: now also J6.3 (Pin_3)
- net VSYS: now also J4.1 (Pin_1), J6.1 (Pin_1); no longer J5.4 (Pin_4)
Other:
- note added: "(Optional) Pull-up resistor for I2C (GPIO 0,1)"
- note added: "Pin holes"
- note added: "Test pads for debug ports"
- note removed: "BOOTSEL"
- note removed: "Reset"
- moved on the sheet: J1, J2, J3, R2, R6

Commit message: v0.2
Parts:
- removed J1: FFC connector, ec_parts:HRS_FH34SRJ-08S-0.5SH(50), symbol Connector_Generic_MountingPin:Conn_01x08_MountingPin
- removed J2: Right, ec_parts:Right_PinHeader_1x11_P2.54mm_Vertical, symbol Connector_Generic:Conn_01x11
- removed J3: Bottom pin pads, ec_parts:ec_pad_1x15_P1.27mm, symbol Connector_Generic:Conn_01x15
- removed J4: Left, ec_parts:Left_PinHeader_1x12_P2.54mm_Vertical, symbol Connector_Generic:Conn_01x12
- removed J5: Conn_01x04, ec_parts:TestPinHeader_1x03_P1.27mm_Vertical, symbol Connector_Generic:Conn_01x03
- removed J6: Molex Pico Ezmate 1x04 or 1x06, ec_parts:Molex_Pico-EZmate_1.2mm_04_or_06, symbol Connector_Generic_MountingPin:Conn_01x06_MountingPin
- removed R2, R6: 27, Resistor_SMD_AKL:R_0603_1608Metric_Pad0.98x0.95mm_HandSolder, symbol Device:R
- added J1: rp2040_controller, ec_parts:rp2040_controller, symbol ec_parts:rp2040_controller
Connections:
- net +3V3: now also J1.16 (GPIO13), J1.18 (GPIO15), J1.30 (GPIO19), J1.7 (GPIO5)
- net GND: now also J1.17 (GPIO14), J1.31 (GPIO20), J1.32 (GPIO21), J1.41 (GPIO29/ADC3)
- net GPIO0: now also J1.5 (GPIO3)
- net GPIO1: now also J1.6 (GPIO4)
- net GPIO10: now also J1.15 (GPIO12)
- net GPIO11: now also J1.19 (TESTEN)
- net GPIO12: now also J1.20 (XIN)
- net GPIO13: now also J1.21 (XOUT)
- net GPIO14: now also J1.22 (IOVDD)
- net GPIO16: now also J1.26 (RUN)
- net GPIO17: now also J1.27 (GPIO16)
- net GPIO18: now also J1.28 (GPIO17)
- net GPIO19: now also J1.29 (GPIO18)
- net GPIO2: now also J1.39 (GPIO27/ADC1)
- net GPIO20: now also J1.33 (IOVDD)
- net GPIO21: now also J1.34 (GPIO22)
- net GPIO22: now also J1.35 (GPIO23)
- net GPIO23: now also J1.36 (GPIO24)
- net GPIO24: now also J1.37 (GPIO25)
- net GPIO26/ADC0: now also J1.25 (SWDIO)
- net GPIO27/ADC1: now also J1.24 (SWCLK)
- net GPIO28/ADC2: now also J1.23 (DVDD)
- net GPIO3: now also J1.9 (GPIO7)
- net GPIO4: now also J1.38 (GPIO26/ADC0)
- net GPIO5: now also J1.10 (IOVDD)
- net GPIO6: now also J1.11 (GPIO8)
- net GPIO7: now also J1.12 (GPIO9)
- net GPIO8: now also J1.13 (GPIO10)
- net GPIO9: now also J1.14 (GPIO11)
- net RUN: now also J1.40 (GPIO28/ADC2)
- net SWCLK: now also J1.1 (IOVDD)
- net SWDIO: now also J1.42 (IOVDD)
- net USB_BOOT: now also J1.8 (GPIO6)
- net USB_N: now also J1.3 (GPIO1)
- net USB_P: now also J1.4 (GPIO2)
- net VSYS: now also J1.2 (GPIO0)
Other:
- note added: "Pin holes mill-max socket for side : 0305-1, 7305-0, 3305-0"
- note removed: "(Optional) Pull-up resistor for I2C (GPIO 0,1)"
- note removed: "Pin holes"
- note removed: "Test pads for debug ports"

Commit message: v0.3
Parts:
- removed U2: AP2112K-3.3TRG1, ap2112:AP2112K-3.3TRG1, symbol rpi-pico-debugger-shoe-rescue:AP2112K-3.3TRG1-2021-05-12_00-19-53
- added R2: 400, Resistor_SMD_AKL:R_0603_1608Metric_Pad0.98x0.95mm_HandSolder, symbol Device:R
- added U2: AP2112K-3.3, Package_TO_SOT_SMD_AKL:SOT-23-5, symbol Regulator_Linear:AP2112K-3.3
Connections:
- net +3V3: now also J1.9 (GPIO7), R2.2, U2.5 (VOUT); no longer C8.1, J1.7 (GPIO5), U1.43 (ADC_AVDD)
- net GND: now also J1.39 (GPIO27/ADC1), U2.2 (GND); no longer J1.41 (GPIO29/ADC3), Y1.2
- net GPIO2: now also J1.40 (GPIO28/ADC2); no longer J1.39 (GPIO27/ADC1)
- net GPIO3: now also J1.8 (GPIO6); no longer J1.9 (GPIO7)
- net RUN: now also J1.41 (GPIO29/ADC3); no longer J1.40 (GPIO28/ADC2)
- net USB_BOOT: now also J1.7 (GPIO5); no longer J1.8 (GPIO6)
- net VSYS: now also U2.1 (VIN)
- net at R3.2: now also U2.3 (EN)
- new net AVDD: C8.1, R2.1, U1.43 (ADC_AVDD)
- no-connect marks 1 -> 0
Other:
- moved on the sheet: C11, C13, C14, C15, C6, C9, R3, Y1

Commit message: temp
Parts:
- removed J1: rp2040_controller, ec_parts:rp2040_controller, symbol ec_parts:rp2040_controller
- added J1, J3: Conn_01x12, ec_parts:PinHeader_1x12_P2.54mm_Vertical, symbol Connector_Generic:Conn_01x11
- added J2: Conn_01x15, ec_parts:PinHeader_1x15_P1.27mm_Vertical, symbol Connector_Generic:Conn_01x15
- added J4: Conn_01x05, ec_parts:TestPinHeader_1x03_P1.27mm_Vertical, symbol Connector_Generic:Conn_01x03
- added J5, J6: Conn_01x02, Connector_PinHeader_2.54mm:PinHeader_1x02_P2.54mm_Vertical, symbol Connector_Generic:Conn_01x02
- added J?: rp2040_controller, ec_parts:ec_pad_1x15_P1.27mm, symbol ec_parts:rp2040_controller
Connections:
- net +3V3: now also J2.14 (Pin_14), J2.2 (Pin_2), J3.4 (Pin_4)
- net GND: now also J1.4 (Pin_4), J2.1 (Pin_1), J2.15 (Pin_15), J3.1 (Pin_1)
- net GPIO10: now also J3.11 (Pin_11)
- net GPIO11: now also J2.13 (Pin_13)
- net GPIO12: now also J2.12 (Pin_12)
- net GPIO13: now also J2.11 (Pin_11)
- net GPIO14: now also J2.10 (Pin_10)
- net GPIO16: now also J2.6 (Pin_6)
- net GPIO17: now also J2.5 (Pin_5)
- net GPIO18: now also J2.4 (Pin_4)
- net GPIO19: now also J2.3 (Pin_3)
- net GPIO20: now also J1.11 (Pin_11)
- net GPIO21: now also J1.10 (Pin_10)
- net GPIO22: now also J1.9 (Pin_9)
- net GPIO23: now also J1.8 (Pin_8)
- net GPIO24: now also J1.7 (Pin_7)
- net GPIO25: now also J1.2 (Pin_2)
- net GPIO26/ADC0: now also J2.7 (Pin_7)
- net GPIO27/ADC1: now also J2.8 (Pin_8)
- net GPIO28/ADC2: now also J2.9 (Pin_9)
- net GPIO29/ADC3: now also J3.2 (Pin_2)
- net GPIO8: now also J3.9 (Pin_9)
- net GPIO9: now also J3.10 (Pin_10)
- net RUN: now also J1.3 (Pin_3)
- net SWCLK: now also J4.1 (Pin_1)
- net SWDIO: now also J4.2 (Pin_2)
- net USB_BOOT: now also J3.3 (Pin_3)
- net USB_N: now also J5.1 (Pin_1)
- net USB_P: now also J6.2 (Pin_2)
- net VSYS: now also J1.1 (Pin_1)
- net GPIO0 renamed GPIO0/I2C0_SDA
- net GPIO0/I2C0_SDA: now also J5.2 (Pin_2)
- net GPIO1 renamed GPIO1/I2C0_SCL
- net GPIO1/I2C0_SCL: now also J6.1 (Pin_1)
- net GPIO2 renamed GP_2/I2C_1_SDA/SPI_0_SCK
- net GP_2/I2C_1_SDA/SPI_0_SCK: now also J1.5 (Pin_5)
- net GPIO3 renamed GP_3/I2C_1_SCL/SPI_0_TX 
- net GP_3/I2C_1_SCL/SPI_0_TX : now also J3.5 (Pin_5)
- net GPIO4 renamed GP_4/I2C_0_SDA/SPI_0_RX
- net GP_4/I2C_0_SDA/SPI_0_RX: now also J1.6 (Pin_6)
- net GPIO5 renamed GP_5/I2C_0_SCL/SPI_0_CS
- net GP_5/I2C_0_SCL/SPI_0_CS: now also J3.6 (Pin_6)
- net GPIO6 renamed GP_6/I2C_1_SDA/SPI_0_SCK
- net GP_6/I2C_1_SDA/SPI_0_SCK: now also J3.7 (Pin_7)
- net GPIO7 renamed GP_7/I2C_1_SCL/SPI_0_TX
- net GP_7/I2C_1_SCL/SPI_0_TX: now also J3.8 (Pin_8)
