File: rp2040_controller.kicad_sch (KiCad schematic)
At the start: 28 parts, among them J7 rp2040_controller, U1 RP2040, U2 AP2112K-3.3, U3 W25Q64JV, Y1 XYDBPCNANF-12MHZ

Commit message: Kicad 7
Parts:
- removed U1: RP2040, rp2040:RP2040, symbol rpi-pico-debugger-shoe-rescue:RP2040-2021-05-11_23-45-12
- added U1: RP2040, Package_DFN_QFN:QFN-56-1EP_7x7mm_P0.4mm_EP3.2x3.2mm, symbol MCU_RaspberryPi:RP2040
- C1, C10, C11, C12, C13, C14, C15, C16, C2, C3, C4, C5, C6, C7, C8, C9: footprint Capacitor_SMD_AKL:C_0603_1608Metric_Pad1.08x0.95mm -> PCM_Capacitor_SMD_AKL:C_0603_1608Metric_Pad1.08x0.95mm
- R1, R2, R3, R4, R5, R8, R9: footprint Resistor_SMD_AKL:R_0603_1608Metric_Pad0.98x0.95mm_HandSolder -> PCM_Resistor_SMD_AKL:R_0603_1608Metric_Pad0.98x0.95mm_HandSolder
- U2: footprint Package_TO_SOT_SMD_AKL:SOT-23-5 -> PCM_Package_TO_SOT_SMD_AKL:SOT-23-5
- U3: footprint Package_SON:WSON-8-1EP_6x5mm_P1.27mm_EP3.4x4mm -> PCM_Package_SON_AKL:WSON-8-1EP_6x5mm_P1.27mm_EP3.4x4mm
- Y1: footprint Crystal_AKL:Crystal_SMD_2520-4Pin_2.5x2.0mm -> PCM_Crystal_AKL:Crystal_SMD_2520-4Pin_2.5x2.0mm
- renumbered J7 to J1
Connections:
- net +1.1V: now also U1.23 (DVDD), U1.45 (VREG_VOUT), U1.50 (DVDD)
- net +3V3: now also U1.1 (IOVDD), U1.10 (IOVDD), U1.22 (IOVDD), U1.33 (IOVDD), U1.42 (IOVDD), U1.44 (VREG_IN), U1.48 (USB_VDD), U1.49 (IOVDD)
- net AVDD: now also U1.43 (ADC_AVDD)
- net GND: now also Y1.2, U1.19 (TESTEN), U1.57 (GND)
- net GPIO0/I2C0_SDA: now also U1.2 (GPIO0)
- net GPIO10: now also U1.13 (GPIO10)
- net GPIO11: now also U1.14 (GPIO11)
- net GPIO12: now also U1.15 (GPIO12)
- net GPIO13: now also U1.16 (GPIO13)
- net GPIO14: now also U1.17 (GPIO14)
- net GPIO15: now also U1.18 (GPIO15)
- net GPIO16: now also U1.27 (GPIO16)
- net GPIO17: now also U1.28 (GPIO17)
- net GPIO18: now also U1.29 (GPIO18)
- net GPIO19: now also U1.30 (GPIO19)
- net GPIO1/I2C0_SCL: now also U1.3 (GPIO1)
- net GPIO20: now also U1.31 (GPIO20)
- net GPIO21: now also U1.32 (GPIO21)
- net GPIO22: now also U1.34 (GPIO22)
- net GPIO23: now also U1.35 (GPIO23)
- net GPIO24: now also U1.36 (GPIO24)
- net GPIO25: now also U1.37 (GPIO25)
- net GPIO26/ADC0: now also U1.38 (GPIO26_ADC0)
- net GPIO27/ADC1: now also U1.39 (GPIO27_ADC1)
- net GPIO28/ADC2: now also U1.40 (GPIO28_ADC2)
- net GPIO29/ADC3: now also U1.41 (GPIO29_ADC3)
- net GPIO8: now also U1.11 (GPIO8)
- net GPIO9: now also U1.12 (GPIO9)
- net GP_2/I2C_1_SDA/SPI_0_SCK: now also U1.4 (GPIO2)
- net GP_3/I2C_1_SCL/SPI_0_TX : now also U1.5 (GPIO3)
- net GP_4/I2C_0_SDA/SPI_0_RX: now also U1.6 (GPIO4)
- net GP_5/I2C_0_SCL/SPI_0_CS: now also U1.7 (GPIO5)
- net GP_6/I2C_1_SDA/SPI_0_SCK: now also U1.8 (GPIO6)
- net GP_7/I2C_1_SCL/SPI_0_TX: now also U1.9 (GPIO7)
- net QSPI_CS: now also U1.56 (QSPI_SS)
- net QSPI_SCK: now also U1.52 (QSPI_SCLK)
- net QSPI_SD0: now also U1.53 (QSPI_SD0)
- net QSPI_SD1: now also U1.55 (QSPI_SD1)
- net QSPI_SD2: now also U1.54 (QSPI_SD2)
- net QSPI_SD3: now also U1.51 (QSPI_SD3)
- net RUN: now also U1.26 (RUN)
- net SWCLK: now also U1.24 (SWCLK)
- net SWDIO: now also U1.25 (SWD)
- net at R5.2: now also U1.46 (USB_DM)
- net at R4.2: now also U1.47 (USB_DP)
- net USB_N renamed DM
- net USB_P renamed DP
- net XIN: no longer names the net of C13.1, Y1.3
- net XIN: now also U1.20 (XIN)
- net XOUT: no longer names the net of C15.1, Y1.1
- net XOUT: now also U1.21 (XOUT)
Other:
- note added: "DVDD pin capacitors"
- note added: "IOVDD pin capacitors"
- note removed: "Buttons"
- note removed: "Close to ADC_AVDD"
- note removed: "Each close to a DVDD pin"
- note removed: "Each close to an IOVDD pin"
- note removed: "Microcontroller"
- note removed: "Optional Connectors"
- note removed: "Target Connector"
- note removed: "USB and Power"
- moved on the sheet: C1, C11, C13, C14, C15, C16, C2, C3, C4, C5, C6, C7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
